File: sensor_PCB_KiCad/Untitled/Untitled.kicad_pcb (KiCad board)
At the start: 2 copper layers, 38 x 10 mm, 7 parts, among them U1 DRV5055A3xDBZxQ1, U2 DRV5055A3xDBZxQ1, U3 DRV5055A3xDBZxQ1

Commit message: added latest changes
Parts:
- HE0: renamed from U1; value DRV5055A3xDBZxQ1 -> ADC 0
- HE1: renamed from U2; value DRV5055A3xDBZxQ1 -> ADC 1
- HE2: renamed from U3; value DRV5055A3xDBZxQ1 -> ADC 2
- renumbered C3 to C0, C2 to C1, C1 to C2
Changed lines of the file:
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@@
 		(descr "SOT, 3 Pin (https://www.jedec.org/system/files/docs/to-236h.pdf variant AB), generated with kicad-footprint-generator ipc_gullwing_generator.py")
 		(tags "SOT TO_SOT_SMD")
-		(property "Reference" "U2"
-			(at 0 -2.4 90)
-			(layer "F.SilkS")
-			(effects
-				(font
-					(size 1 1)
-					(thickness 0.15)
-				)
-			)
-		)
-		(property "Value" "DRV5055A3xDBZxQ1"
+		(property "Reference" "HE1"
+			(at 2.95 0 0)
+			(layer "F.SilkS")
+			(effects
+				(font
+					(size 1 1)
+					(thickness 0.15)
+				)
+			)
+		)
+		(property "Value" "ADC 1"
 			(at 0 2.4 90)
 			(layer "F.Fab")
@@
 		(descr "Capacitor SMD 0603 (1608 Metric), square (rectangular) end terminal, IPC_7351 nominal, (Body size source: IPC-SM-782 page 76, https://www.pcb-3d.com/wordpress/wp-content/uploads/ipc-sm-782a_amendment_1_and_2.pdf), generated with kicad-footprint-generator")
 		(tags "capacitor")
-		(property "Reference" "C3"
-			(at 0 -1.43 90)
+		(property "Reference" "C0"
+			(at -0.475 -1.9 0)
 			(layer "F.SilkS")
 			(effects
@@
 		)
 		(property "Value" "0.01u"
-			(at 0 1.43 90)
+			(at 1.225 2.8 90)
 			(layer "F.Fab")
 			(effects
@@
 		(descr "Capacitor SMD 0603 (1608 Metric), square (rectangular) end terminal, IPC_7351 nominal, (Body size source: IPC-SM-782 page 76, https://www.pcb-3d.com/wordpress/wp-content/uploads/ipc-sm-782a_amendment_1_and_2.pdf), generated with kicad-footprint-generator")
 		(tags "capacitor")
-		(property "Reference" "C1"
-			(at 0 -1.43 -90)
+		(property "Reference" "C2"
+			(at 0.075 -2.15 0)
 			(layer "F.SilkS")
 			(effects
@@
 		)
 		(property "Value" "0.01u"
-			(at 0 1.43 -90)
+			(at 0.925 -3.9 90)
 			(layer "F.Fab")
 			(effects
@@
 		)
 		(fp_text user "${REFERENCE}"
-			(at 0 0 -90)
+			(at 0 0 90)
 			(layer "F.Fab")
 			(effects
@@
 		(descr "SOT, 3 Pin (https://www.jedec.org/system/files/docs/to-236h.pdf variant AB), generated with kicad-footprint-generator ipc_gullwing_generator.py")
 		(tags "SOT TO_SOT_SMD")
-		(property "Reference" "U3"
-			(at 0 -2.4 90)
-			(layer "F.SilkS")
-			(effects
-				(font
-					(size 1 1)
-					(thickness 0.15)
-				)
-			)
-		)
-		(property "Value" "DRV5055A3xDBZxQ1"
+		(property "Reference" "HE2"
+			(at 2.95 0 0)
+			(layer "F.SilkS")
+			(effects
+				(font
+					(size 1 1)
+					(thickness 0.15)
+				)
+			)
+		)
+		(property "Value" "ADC 2"
 			(at 0 2.4 90)
 			(layer "F.Fab")
@@
 		(descr "Capacitor SMD 0603 (1608 Metric), square (rectangular) end terminal, IPC_7351 nominal, (Body size source: IPC-SM-782 page 76, https://www.pcb-3d.com/wordpress/wp-content/uploads/ipc-sm-782a_amendment_1_and_2.pdf), generated with kicad-footprint-generator")
 		(tags "capacitor")
-		(property "Reference" "C2"
-			(at 0 -1.43 90)
+		(property "Reference" "C1"
+			(at 0.1 -2.1 0)
 			(layer "F.SilkS")
 			(effects
@@
 		)
 		(property "Value" "0.01u"
-			(at 0 1.43 90)
+			(at 1.2 -3.85 90)
 			(layer "F.Fab")
 			(effects
@@
 			(unlocked yes)
 			(layer "F.SilkS")
+			(hide yes)
 			(effects
 				(font
@@
 		(descr "SOT, 3 Pin (https://www.jedec.org/system/files/docs/to-236h.pdf variant AB), generated with kicad-footprint-generator ipc_gullwing_generator.py")
 		(tags "SOT TO_SOT_SMD")
-		(property "Reference" "U1"
-			(at 0 -2.4 90)
-			(layer "F.SilkS")
-			(effects
-				(font
-					(size 1 1)
-					(thickness 0.15)
-				)
-			)
-		)
-		(property "Value" "DRV5055A3xDBZxQ1"
+		(property "Reference" "HE0"
+			(at 3 0 0)
+			(layer "F.SilkS")
+			(effects
+				(font
+					(size 1 1)
+					(thickness 0.15)
+				)
+			)
+		)
+		(property "Value" "ADC 0"
 			(at 0 2.4 90)
 			(layer "F.Fab")
-			(effects
-				(font
+			(hide yes)
+			(effects
+				(font
